File: Badge_RP2350_FPGA/Badge_RP2350_FPGA.kicad_pcb (KiCad board)
At the start: 2 copper layers, 100 x 150 mm, 103 parts, among them J1 USB_C_Receptacle_USB2.0_16P, J2 Conn_01x03_Pin, J3 Conn_01x15_Pin, J4 Conn_01x15_Pin, SW1 SW_Push, SW12 On/Off, SW2 SW_Push, U1 RP2350_60QFN, U2 GW1N-LV9QN88C6_I5_, U3 ME6211C12, U4 TMI7003C, U6 W25Q32JVSS, U7 W25Q32JVSS, U8 TPS61221DCK, Y1 ABM8-272-T3

Commit message: put pull up to mode1, pull down to mode0
Parts:
- added R23: 1K, Resistor_SMD:R_0402_1005Metric, F.Cu at (114.8, 128.1)
- added R24: 4.7K, Resistor_SMD:R_0402_1005Metric, F.Cu at (111.2, 137.0)
Connections:
- J4 pad 14: T8A -> unconnected-(J4-Pin_14-Pad14)
- J4 pad 15: T8B -> unconnected-(J4-Pin_15-Pad15)
- U2 pad 85: T8B -> unconnected-(U2-IOT8B-Pad85)
- U2 pad 86: T8A -> unconnected-(U2-IOT8A-Pad86)
Routing:
- net T8A: track 50.0 -> 0.00 mm, vias 1 -> 0
- net T8B: track 48.3 -> 0.00 mm, vias 1 -> 0
- net VCC03_1V8: track 53.6 -> 56.1 mm
- net MODE1: track 51.1 -> 52.7 mm, vias 1 -> 2
- net MODE0: track 52.3 -> 53.5 mm, vias 1 -> 2
- net COL1: track 116.8 -> 117.5 mm
- net GND: vias 173 -> 176
Other:
- board text removed: "T8A"
- board text removed: "T8B"
