File: Badge_RP2350_FPGA/power_delivery_sch.kicad_sch (KiCad schematic)
At the start: 28 parts, among them J1 USB_C_Receptacle_USB2.0_16P, SW12 On/Off, U3 ME6211C12, U4 TMI7003C

Commit message: Version 1.6: fix FB3 error, fix missing secondary flash pull-up, fix missing diode on battery, realign and add silkscreen
Parts:
- added D4: D_Schottky, Diode_SMD:D_SOD-123, symbol Device:D_Schottky
Connections:
- net GND: now also C42.2, R16.2; no longer C5.2, R1.2, R16.1, U4.2 (FB3)
- net VBUS: now also D4.1 (K); no longer SW12.3 (C)
- new net: D4.2 (A), SW12.3 (C)
- new net: C5.2, R1.2, R16.1, U4.2 (FB3)
Other:
- moved on the sheet: C42, C5, R1, R16

Commit message: fix power boost issue
Parts:
- added U8: TPS61221DCK, Package_TO_SOT_SMD:Texas_R-PDSO-G6, symbol Regulator_Switching:TPS61221DCK
Connections:
- net GND: now also U8.3 (GND)
- net VBUS: now also U8.2 (FB), U8.4 (VOUT); no longer D4.1 (K)
- new net: D4.1 (K), U8.1 (VIN), U8.6 (EN)
